File: PCB/ESC_Device_Hub_v0/ESC_Device_Hub_v0.kicad_sch (KiCad schematic)
At the start: 135 parts, among them J1 Conn_01x04, J10 Conn_01x06, J11 Conn_01x02, J12 Conn_01x02, J13 Conn_01x02, J14 Conn_01x02, J15 Conn_01x02, J16 Conn_01x02, J17 Conn_01x02, J18 Conn_01x02, J19 Conn_01x05, J2 Conn_01x04, J20 Conn_01x01, J21 Conn_01x01, J22 Conn_01x02, J3 Conn_01x04, J4 Conn_01x04, J5 Conn_01x04, J6 Conn_01x04, J7 Conn_01x06, J8 Conn_01x06, J9 Conn_01x06, SW1 SW_Push, SW2 SW_Push, SW3 SW_Coded_SH-7050, SW4 SW_DIP_x02, U1 ISO1042BQDWVRQ1, U18 USB_Type-C, U2 MCP2562FD-H/MF, U3 IS25LP064D-JLLE, U4 STM32H563RGVx, U5 NJW1933F1-AT, U6 TLP293, U7 NJM2884U1-33, U8 XC8114AA01PR-G, U9 XC8114AA01PR-G, Y1 FC2012SN 32.768K-70NNA0KC0

Commit message: PCB作成残りGNDのビア打ちをきちんとやるだけ
Parts:
- added C33: 0.1uF, Capacitor_SMD:C_0402_1005Metric_Pad0.74x0.62mm_HandSolder, symbol Device:C_Small
- added R24: 10k, Resistor_SMD:R_0402_1005Metric_Pad0.72x0.64mm_HandSolder, symbol Device:R_Small
- C10, C11, C3, C5, C6: footprint Capacitor_SMD:C_0603_1608Metric_Pad1.08x0.95mm_HandSolder -> Capacitor_SMD:C_0402_1005Metric_Pad0.74x0.62mm_HandSolder
- C28: value 0.1uF -> 2.2uF
- U1: value ISO1042BQDWVRQ1 -> ISO1042BQDWVQ1
- U17: value ~ -> (none)
Connections:
- net +3.3V: now also R24.1
- net +5VA: now also U9.3 (EN); no longer U9.2 (EP)
- net FLASH_SS: now also R24.2
- net GND: now also U8.2 (EP), U9.2 (EP), C33.2; no longer U8.3 (EP), U9.3 (EP)
- net LED_1: now also U4.59 (PB5); no longer U4.27 (PB1)
- net LED_2: now also U4.56 (PC12); no longer U4.28 (PB2)
- net LED_3: now also U4.55 (PC11); no longer U4.57 (PB3(JTDO)
- net LED_4: now also U4.54 (PC10); no longer U4.58 (PB4(NJTRST))
- net LIMS2_1: now also U4.26 (PB0); no longer U4.40 (PC6)
- net LIMS2_2: now also U4.27 (PB1); no longer U4.41 (PC7)
- net LIMS3_1: now also U4.28 (PB2); no longer U4.42 (PC8)
- net LIMS3_2: now also U4.30 (PB11); no longer U4.43 (PC9)
- net LIMS4_1: now also D23.1 (K), J17.2 (Pin_2), R60.1, U4.36 (PB14); no longer D26.1 (K), J18.2 (Pin_2), R66.1, U4.55 (PC11)
- net LIMS4_2: now also D26.1 (K), J18.2 (Pin_2), R66.1, U4.37 (PB15); no longer D23.1 (K), J17.2 (Pin_2), R60.1, U4.54 (PC10)
- net NRST: now also C33.1
- net POWER_MONITOR: now also U4.2 (PC13); no longer U4.26 (PB0)
- net Rol_SW1: now also U4.40 (PC6); no longer U4.36 (PB14)
- net Rol_SW2: now also U4.41 (PC7); no longer U4.37 (PB15)
- net Rol_SW4: now also U4.42 (PC8); no longer U4.38 (PD11)
- net Rol_SW8: now also U4.43 (PC9); no longer U4.39 (PD12)
- net Synchronization_Enable: now also U4.39 (PD12)
- net Synchronization_Master: now also U4.38 (PD11)
- net at C12.1, FB1.2, U8.4 (Vin): now also U8.3 (EN); no longer U8.2 (EP)
- no-connect marks 4 -> 9
Other:
- note added: "ESC-Control-Hub_v0"
- moved on the sheet: C12, C13, C3, C32, C4, C5, J19, JP2, R1, U2, U8
Changed lines of the file:
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@@
 (kicad_sch
-	(version 20250114)
+	(version 20260306)
 	(generator "eeschema")
-	(generator_version "9.0")
+	(generator_version "10.0")
 	(paper "A3")
