File: PCB/ESC_Device_Hub_v1/ESC_Device_Hub_v1.kicad_pcb (KiCad board)
At the start: 4 copper layers, 50 x 90 mm, 144 parts, among them J1 Conn_01x04, J10 Conn_01x06, J11 Conn_01x02, J12 Conn_01x02, J13 Conn_01x02, J14 Conn_01x02, J15 Conn_01x02, J16 Conn_01x02, J17 Conn_01x02, J18 Conn_01x02, J19 Conn_01x05, J2 Conn_01x04, J20 Conn_01x01, J21 Conn_01x01, J22 Conn_01x02, J3 Conn_01x04, J4 Conn_01x04, J5 Conn_01x04, J6 Conn_01x04, J7 Conn_01x06, J8 Conn_01x06, J9 Conn_01x06, SW1 SW_Push, SW2 SW_Push, SW3 SW_Coded_SH-7050, SW4 SW_DIP_x02, U1 ISO1042BQDWVQ1, U10 LM66100DCK, U11 LM66100DCK, U18 USB_Type-C, U2 MCP2562FD-H/MF, U3 IS25LP064D-JLLE, U4 STM32H563RGVx, U5 NJW1933F1-AT, U6 TLP293, U7 NJM2884U1-33, Y1 FC2012SN 32.768K-70NNA0KC0, Y2 XRCGB25M000FFS1AR0

Commit message: MCUの向き決定 LSE HSE配置
Parts:
- moved R1 101.1 mm to (144.3, 38.7)
- moved C34 81.0 mm to (153.6, 51.8), turned to 180 degrees
- moved C30 80.9 mm to (154.2, 50.4), turned to 180 degrees
- moved C31 80.4 mm to (154.2, 49.5), turned to 180 degrees
- moved U3 79.5 mm to (166.9, 66.1), turned to 180 degrees
- moved C35 79.3 mm to (155.2, 53.1), turned to -90 degrees
- moved C21 76.5 mm to (155.5, 48.6), turned to 180 degrees
- moved C22 75.9 mm to (155.5, 47.7), turned to 180 degrees
- moved J19 74.4 mm to (137.1, 64.2), turned to -90 degrees
- moved C19 70.1 mm to (157.0, 46.9), turned to 90 degrees
- moved Y1 69.5 mm to (152.1, 50.0), turned to 90 degrees
- moved JP2 68.7 mm to (145.4, 41.6), turned to -90 degrees
- moved Y2 67.7 mm to (153.6, 53.2)
- moved U2 58.8 mm to (164.0, 36.6), turned to 180 degrees
- moved U18 43.8 mm to (187.2, 43.0), turned to 90 degrees
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Routing:
- net XTAL_IN: track 0.00 -> 5.52 mm
- net XTAL_OUT: track 0.00 -> 5.31 mm
- net HSE_IN: track 0.00 -> 4.73 mm
- net USB_DFU_DP: track 0.00 -> 4.28 mm
- net FLASH_IO1: track 0.00 -> 4.20 mm
- net USB_DFU_DM: track 0.00 -> 4.19 mm
- net FLASH_IO3: track 0.00 -> 4.12 mm
- net FLASH_IO2: track 0.00 -> 4.11 mm
- net FLASH_IO0: track 0.00 -> 4.11 mm
- net FLASH_SS: track 0.00 -> 4.06 mm
- net +3.3V: track 0.00 -> 3.87 mm
- net FLASH_SCK: track 0.00 -> 3.87 mm
- net HSE_OUT: track 0.00 -> 3.75 mm
- net FDCAN_RXD: track 0.00 -> 3.12 mm
- net ESC_FDCAN_RXD: track 0.00 -> 2.95 mm
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
Commit message: QuadSPI周りのピンの使用禁止
Parts:
- C16, C18, C23, C24: moved to B.Cu
- moved C23 76.2 mm to (156.0, 53.8), turned to 90 degrees
- moved C24 74.9 mm to (156.9, 53.8), turned to 90 degrees
- moved C16 71.8 mm to (157.5, 56.5)
- moved C18 62.7 mm to (164.7, 49.4), turned to -90 degrees
Routing:
- net GND: track 0.00 -> 11.4 mm
- net +3.3V: track 3.87 -> 8.49 mm, vias 0 -> 3
