File: PCB/ESC_Device_Hub_v1/ESC_Device_Hub_v1.kicad_pcb (KiCad board)
At the start: 4 copper layers, 50 x 90 mm, 137 parts, among them J1 Conn_01x04, J10 Conn_01x06, J11 Conn_01x02, J12 Conn_01x02, J13 Conn_01x02, J14 Conn_01x02, J15 Conn_01x02, J16 Conn_01x02, J17 Conn_01x02, J18 Conn_01x02, J19 Conn_01x05, J2 Conn_01x04, J20 Conn_01x01, J21 Conn_01x01, J22 Conn_01x02, J3 Conn_01x04, J4 Conn_01x04, J5 Conn_01x04, J6 Conn_01x04, J7 Conn_01x06, J8 Conn_01x06, J9 Conn_01x06, SW1 SW_Push, SW2 SW_Push, SW3 SW_Coded_SH-7050, U1 ISO1042BQDWVQ1, U10 LM66100DCK, U11 LM66100DCK, U18 USB_Type-C, U2 MCP2562FD-H/MF, U3 IS25LP064D-JLLE, U4 STM32H563RGVx, U6 TLP293, U7 NJM2884U1-33, U8 RFM-0505S, Y1 FC2012SN 32.768K-70NNA0KC0, Y2 XRCGB25M000FFS1AR0

Commit message: PCB変更
Routing:
- net LIMS3_1: track 74.1 -> 76.0 mm, vias 2 -> 3
- net NRST: track 58.4 -> 59.9 mm
- net POWER_MONITOR: track 62.3 -> 63.4 mm
- net Rol_SW4: track 21.9 -> 21.2 mm
- net +5VA: track 100.9 -> 101.6 mm
- net LIMS2_1: track 63.5 -> 64.1 mm, vias 2 -> 3
- net LIMS4_2: track 71.3 -> 71.5 mm, vias 2 -> 3
- net LIMS3_2: track 60.4 -> 60.6 mm, vias 2 -> 3
- net LIMS2_2: track 49.9 -> 49.7 mm, vias 2 -> 3
- net GNDD: vias 21 -> 219
- net GND: vias 81 -> 481
