File: PCB/ESC_Device_Hub_v1/ESC_Device_Hub_v1.kicad_sch (KiCad schematic)
At the start: 134 parts, among them J1 Conn_01x04, J10 Conn_01x06, J11 Conn_01x02, J12 Conn_01x02, J13 Conn_01x02, J14 Conn_01x02, J15 Conn_01x02, J16 Conn_01x02, J17 Conn_01x02, J18 Conn_01x02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

Commit message: DRC OK残りシルク
Connections:
- net +5VP: no longer J3.3 (Pin_3), J4.3 (Pin_3), J5.3 (Pin_3), J6.3 (Pin_3)
- no-connect marks 8 -> 12

Commit message: PCBできたけどガーバーが出力できない
Connections:
- net GNDD: now also J3.3 (Pin_3), J4.3 (Pin_3), J5.3 (Pin_3), J6.3 (Pin_3)
- no-connect marks 12 -> 8
