File: PCB/ESC_Device_Hub_v1/ESC_Device_Hub_v1.kicad_sch (KiCad schematic)
At the start: 133 parts, among them J1 Conn_01x04, J10 Conn_01x06, J11 Conn_01x02, J12 Conn_01x02, J13 Conn_01x02, J14 Conn_01x02, J15 Conn_01x02, J16 Conn_01x02, J17 Conn_01x02, J18 Conn_01x02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

Commit message: 変更3
Connections:
- net +3.3V: now also C2.1, U1.1 (VCC1)
- net +5V: no longer C2.1, U1.1 (VCC1)
